File: kicad/zed-f9p-dual-adapter.kicad_pcb (KiCad board)
At the start: 4 copper layers, 67.5 x 31.8 mm, 34 parts, among them J1 USB_C_Receptacle_USB2.0_14P, J2 Conn_02x04_Odd_Even, J3 Conn_02x03_Odd_Even, J4 DE9_Socket, U1 CP2102N-Axx-xQFN28, U2 USBLC6-2SC6, U3 MAX3232, U4 AMS1117-3.3

Commit message: Add files via upload
Updated layout to improve manufacturability
Parts:
- D2, D3, D4: footprint LED_SMD:LED_0402_1005Metric -> LED_SMD:LED_0603_1608Metric
- moved D2 0.62 mm to (137.1, 121.0)
- moved D3 0.62 mm to (139.6, 121.0)
- moved R6 0.62 mm to (137.1, 123.5)
- moved R7 0.62 mm to (139.6, 123.5)
Routing:
- net GND: track 29.8 -> 30.6 mm
- net /USB_D-: track 8.75 -> 9.32 mm
